File: coqui-v1.0.brd (EAGLE design)
At the start: 52.7 x 50.2 mm, 32 parts, among them IC1 OPAMP-DUALU, IC3 MCP73831, IC4 MCP1700-33, J1 AYZ0202, X1 USBSMD

Commit message: update
Parts:
- added CA-TUNE: (no value), rcl:CTRIMTZBX4
- moved CAN 3.64 mm to (2.29, 33.5), turned to 180 degrees
Connections:
- net GND: now also CA-TUNE.1
- net N$11: now also CA-TUNE.2
Routing:
- net VBAT: track 54.5 -> 80.6 mm, vias 3 -> 2
- net N$15: track 62.2 -> 85.2 mm
- net AOUT: track 78.9 -> 96.8 mm
- net N$7: track 56.7 -> 39.2 mm
- net VBUS: track 80.1 -> 63.0 mm, vias 0 -> 2
- net N$16: track 59.5 -> 74.0 mm
- net GND: track 218.7 -> 210.3 mm, vias 2 -> 4
- net VAIN: track 57.7 -> 60.6 mm, vias 1 -> 0
- net N$12: track 50.9 -> 48.9 mm, vias 2 -> 0
- net BOUT: track 74.9 -> 73.1 mm, vias 1 -> 3
- net N$11: track 70.4 -> 68.9 mm, vias 1 -> 4
- net N$14: track 51.9 -> 53.4 mm, vias 0 -> 2
- net N$23: track 69.0 -> 67.6 mm, vias 1 -> 0
- net N$8: track 45.1 -> 46.1 mm, vias 2 -> 4
- net VCC: track 46.4 -> 47.2 mm
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