File: coqui-v1.0.sch (EAGLE design)
At the start: 32 parts, among them IC1 OPAMP-DUALU, IC3 MCP73831, IC4 MCP1700-33, J1 AYZ0202, X1 USBSMD

Commit message: update
Parts:
- added CA-TUNE: (no value), rcl:C-TRIMMTZBX4
Connections:
- net GND: now also CA-TUNE.E
- net N$11: now also CA-TUNE.A
Changed lines of the file:
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@@
 <setting verticaltext="up"/>
 </settings>
-<grid distance="0.05" unitdist="inch" unit="inch" style="lines" multiple="1" display="no" altdistance="0.01" altunitdist="inch" altunit="inch"/>
+<grid distance="0.1" unitdist="inch" unit="inch" style="lines" multiple="1" display="no" altdistance="0.01" altunitdist="inch" altunit="inch"/>
 <layers>
 <layer number="1" name="Top" color="4" fill="1" visible="no" active="no"/>
@@
 <part name="JP2" library="pinhead" deviceset="PINHD-1X5" device=""/>
 <part name="JP5" library="pinhead" deviceset="PINHD-1X5" device=""/>
+<part name="CA-TUNE" library="rcl" deviceset="C-TRIMM" device="TZBX4"/>
 </parts>
 <sheets>
@@
 <instance part="RN2" gate="A" x="-233.68" y="74.93" rot="R180"/>
 <instance part="RN2" gate="B" x="-191.77" y="74.93" rot="R180"/>
-<instance part="RN2" gate="C" x="-207.01" y="86.36" rot="R90"/>
-<instance part="RN2" gate="D" x="-201.93" y="86.36" rot="R90"/>
 <instance part="GND11" gate="1" x="-295.91" y="46.99"/>
 <instance part="CA" gate="G$1" x="-314.96" y="116.84" rot="R270"/>
 <instance part="RVA" gate="G$1" x="-214.63" y="45.72" rot="R90"/>
 <instance part="RVB" gate="G$1" x="-200.66" y="45.72" rot="R90"/>
-<instance part="GND6" gate="1" x="-314.96" y="106.68"/>
+<instance part="GND6" gate="1" x="-325.12" y="106.68"/>
 <instance part="CB" gate="G$1" x="-170.18" y="116.84" rot="R270"/>
 <instance part="GND7" gate="1" x="-170.18" y="100.33"/>
@@
 <instance part="JP2" gate="A" x="-307.34" y="54.61" rot="R180"/>
 <instance part="JP5" gate="A" x="-157.48" y="54.61" rot="R180"/>
+<instance part="CA-TUNE" gate="G$1" x="-314.96" y="129.54" rot="R90"/>
 </instances>
 <busses>
@@
 </segment>
 <segment>
-<pinref part="CA" gate="G$1" pin="1"/>
-<pinref part="GND6" gate="1" pin="GND"/>
-</segment>
-<segment>
 <pinref part="CB" gate="G$1" pin="1"/>
 <pinref part="GND7" gate="1" pin="GND"/>
@@
 <pinref part="JP2" gate="A" pin="1"/>
 <wire x1="-304.8" y1="49.53" x2="-295.91" y2="49.53" width="0.1524" layer="91"/>
+</segment>
+<segment>
+<pinref part="CA" gate="G$1" pin="1"/>
+<pinref part="GND6" gate="1" pin="GND"/>
+<wire x1="-325.12" y1="109.22" x2="-322.58" y2="109.22" width="0.1524" layer="91"/>
+<pinref part="CA-TUNE" gate="G$1" pin="E"/>
+<wire x1="-322.58" y1="109.22" x2="-314.96" y2="109.22" width="0.1524" layer="91"/>
+<wire x1="-317.5" y1="129.54" x2="-322.58" y2="129.54" width="0.1524" layer="91"/>
+<wire x1="-322.58" y1="129.54" x2="-322.58" y2="109.22" width="0.1524" layer="91"/>
+<junction x="-322.58" y="109.22"/>
 </segment>
 </net>
@@
 <wire x1="-265.43" y1="118.11" x2="-265.43" y2="111.76" width="0.1524" layer="91"/>
 <junction x="-265.43" y="111.76"/>
-<wire x1="-287.02" y1="109.22" x2="-312.42" y2="109.22" width="0.1524" layer="91"/>
+<wire x1="-287.02" y1="109.22" x2="-304.8" y2="109.22" width="0.1524" layer="91"/>
 <junction x="-287.02" y="109.22"/>
 <pinref part="CA" gate="G$1" pin="2"/>
-</segment>
-</net>
+<wire x1="-304.8" y1="109.22" x2="-312.42" y2="109.22" width="0.1524" layer="91"/>
+<wire x1="-304.8" y1="109.22" x2="-304.8" y2="129.54" width="0.1524" layer="91"/>
+<pinref part="CA-TUNE" gate="G$1" pin="A"/>
+<wire x1="-304.8" y1="129.54" x2="-309.88" y2="129.54" width="0.1524" layer="91"/>
+<junction x="-304.8" y="109.22"/>
+</segment>
+</net>
