File: coqui-v0.2.brd (EAGLE design)
At the start: 75.8 x 18 mm, 33 parts, among them IC3 MCP73831, IC4 MCP1700-33, J1 AYZ0202

Commit message: update
Connections:
- net THRM: now also SV1.1; no longer SV1.6
- net VCC: now also SV1.6; no longer SV1.1
Routing:
- net N$16: track 44.2 -> 55.2 mm, vias 3 -> 2
- net THRM: track 74.8 -> 65.1 mm, vias 2 -> 0
- net N$8: track 47.4 -> 38.2 mm, vias 2 -> 3
- net N$6: track 57.1 -> 48.6 mm, vias 1 -> 2
- net VCC: track 106.6 -> 100.3 mm, vias 1 -> 2
- net GND: track 126.3 -> 120.7 mm, vias 9 -> 6
- net N$12: track 5.97 -> 9.01 mm, vias 0 -> 2
- net N$17: track 53.9 -> 56.9 mm, vias 5 -> 4
- net AOUT: track 32.2 -> 30.5 mm, vias 1 -> 2
- net N$11: track 34.1 -> 32.8 mm
- net N$2: track 49.1 -> 48.4 mm
