File: coqui-v0.2.sch (EAGLE design)
At the start: 21 parts, among them IC3 MCP73831, IC4 MCP1700-33, J1 AYZ0202, X1 USBSMD

Commit message: update
Parts:
- removed PWR1, PWR3: M02PTH, SparkFun-Connectors:M02PTH
- added CHG: 0805, led:LEDCHIPLED_0805
- added RN1: (no value), resistor-dil:4R-NEXB38V
- added SV3, SV4: (no value), con-lstb:MA03-1
Connections:
- new net N$5: CHG.C
- new net N$8: CHG.A, RN1A.1
- new net VBUS1: RN1A.2
Changed lines of the file:
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@@
 <part name="CB" library="SparkFun-Connectors" deviceset="M02" device="PTH"/>
 <part name="GND7" library="supply1" deviceset="GND" device=""/>
-<part name="PWR1" library="SparkFun-Connectors" deviceset="M02" device="PTH"/>
-<part name="PWR3" library="SparkFun-Connectors" deviceset="M02" device="PTH"/>
 <part name="SV1" library="con-lstb" deviceset="MA03-1" device=""/>
 <part name="PWR2" library="SparkFun-Connectors" deviceset="M02" device="PTH"/>
 <part name="SV2" library="con-lstb" deviceset="MA07-1" device=""/>
 <part name="R1" library="pot" deviceset="TRIM_US-" device="3223W"/>
+<part name="SV3" library="con-lstb" deviceset="MA03-1" device=""/>
+<part name="SV4" library="con-lstb" deviceset="MA03-1" device=""/>
+<part name="CHG" library="led" deviceset="LED" device="CHIPLED_0805" value="0805"/>
+<part name="RN1" library="resistor-dil" deviceset="4R-N" device="EXB38V"/>
 </parts>
 <sheets>
@@
 <instance part="CB" gate="G$1" x="50.8" y="96.52" rot="R270"/>
 <instance part="GND7" gate="1" x="50.8" y="80.01"/>
-<instance part="PWR1" gate="G$1" x="182.88" y="40.64"/>
-<instance part="PWR3" gate="G$1" x="154.94" y="43.18"/>
 <instance part="SV1" gate="G$1" x="177.8" y="22.86"/>
 <instance part="PWR2" gate="G$1" x="172.72" y="53.34"/>
 <instance part="SV2" gate="1" x="236.22" y="27.94"/>
 <instance part="R1" gate="G$1" x="220.98" y="50.8"/>
+<instance part="SV3" gate="G$1" x="193.04" y="25.4"/>
+<instance part="SV4" gate="G$1" x="208.28" y="27.94"/>
+<instance part="CHG" gate="G$1" x="82.55" y="-13.97" smashed="yes"/>
+<instance part="RN1" gate="A" x="82.55" y="-6.35" rot="R90"/>
 </instances>
 <busses>
@@
 </segment>
 </net>
+<net name="VBUS1" class="1">
+<segment>
+<pinref part="RN1" gate="A" pin="2"/>
+<wire x1="82.55" y1="-1.27" x2="86.36" y2="-1.27" width="0.1524" layer="91"/>
+</segment>
+</net>
+<net name="N$5" class="0">
+<segment>
+<wire x1="82.55" y1="-19.05" x2="86.36" y2="-19.05" width="0.1524" layer="91"/>
+<wire x1="86.36" y1="-19.05" x2="86.36" y2="-6.35" width="0.1524" layer="91"/>
+<pinref part="CHG" gate="G$1" pin="C"/>
+</segment>
+</net>
+<net name="N$8" class="0">
+<segment>
+<pinref part="CHG" gate="G$1" pin="A"/>
+<pinref part="RN1" gate="A" pin="1"/>
+</segment>
+</net>

Commit message: update
Parts:
- removed CA, CB, PWR2, RA, RB: M02PTH, SparkFun-Connectors:M02PTH
- removed CAN, CBN: 0.01uF, rcl:C-EUC0805
- removed CHG: 0805, led:LEDCHIPLED_0805
- removed ICA: LM555D, adafruit:LM555D
- removed J-FEMALE: MJ-2135, iPhoneSoftModem:MJ-2135
- removed RC: 22K, adafruit2013:R-US_R0805
- removed RN1: (no value), resistor-dil:4R-NEXB38V
- added C1, C3: .01uF, SparkFun:CAP0402-CAP
- added CHG2: 0805, led:LEDCHIPLED_0805
- added ICB1: LM555D, adafruit:LM555D
- added JP2: AUDIO-JACK3, SparkFun-Connectors:AUDIO-JACK3
- added R2: 22k, SparkFun:RESISTOR0402-RES
- added SV5: (no value), con-lstb:MA07-1
- added SV6: (no value), con-lstb:MA06-1
- added SV7: (no value), con-lstb:MA04-1
- R1: value (none) -> 10k; device pot:TRIM_US-3223W -> SparkFun:RESISTOR0402-RES
- SV2: device con-lstb:MA07-1 -> con-lstb:MA06-1
- SV3, SV4: device con-lstb:MA03-1 -> con-lstb:MA07-1
Connections:
- removed net BOUT: ICA.Q, RB.2
- removed net N$15: CBN.2, ICA.CV
- removed net N$16: CB.2, ICA.THR, ICA.TR, RB.1
- removed net N$6: J-FEMALE.4
- removed net N$8: CHG.A, RN1A.1
- removed net VBIN: ICA.R, ICA.V+
- removed net VBUS1: RN1A.2
- new net AOUT1: ICB1.Q, SV5.3, SV5.7
- new net N$1: ICB1.THR, ICB1.TR, SV5.5, SV5.6
- new net N$2: C1.2, ICB1.CV
- new net N$4: CHG2.A, R1.1
- new net RING1: JP2.RING1
- new net RING2: JP2.RING2
- new net SLEEVE: JP2.EARTH
- new net TIP: JP2.TIP
- new net VAIN1: ICB1.R, ICB1.V+, SV5.2
- net AOUT: now also SV3.3, SV3.7; no longer RA.2
- net GND: now also C1.1, C3.1, ICB1.GND, R2.1, SV1.2, SV1.3, SV3.1, SV3.4, SV5.1, SV5.4; no longer CA.1, CAN.1, CB.1, CBN.1, ICA.GND, RC.1
- net N$11: now also SV3.5, SV3.6; no longer CA.2, RA.1
- net N$14: now also C3.2; no longer CAN.2
- net N$3: now also R2.2; no longer RC.2
- net N$5: now also CHG2.C, IC3.STAT; no longer CHG.C
- net VAIN: now also SV3.2
- net VBUS: now also R1.2
- net VCC: now also SV1.1
- net VDD: now also J1.4
Other:
- moved on the sheet: BATT, IC3, IC4, J1, SV1

Commit message: update
Parts:
- removed C3: .01uF, SparkFun:CAP0402-CAP
- removed SV2: (no value), con-lstb:MA06-1
- removed SV3, SV4, SV5: (no value), con-lstb:MA07-1
- removed X1: USBSMD, SparkFun:USBSMD
- added C2: 0.1uF, SparkFun:CAP0603-CAP
- added CON1, CON2, CON3, CON4: (no value), pinhead:PINHD-1X2
- added D3: SCHOTTKY, adafruit:DIODE_SOD-123FL
- added IN1, IN2, THRM: 1X2-3.5MM, adafruit:1X2-3.5MM
- added JP1: (no value), trrs-dwb:PINHD-1X4/90
- added JP3: (no value), pinhead:PINHD-1X1
- added L1: 500mA, adafruit:PTCFUSE-1206
- added RTHERM: 10k, microbuilder:RESISTOR_0603_NOOUT
- added SV8: (no value), con-lstb:MA06-1
- added U$4: (no value), Testing:USB-AB""
- C1: value .01uF -> 0.1uF; device SparkFun:CAP0402-CAP -> SparkFun:CAP0603-CAP
- R1, R2: device SparkFun:RESISTOR0402-RES -> microbuilder:RESISTOR_0603_NOOUT
- SV1: device con-lstb:MA03-1 -> con-lstb:MA07-1
Connections:
- removed net RING1: JP2.RING1
- removed net RING2: JP2.RING2
- removed net SLEEVE: JP2.EARTH
- removed net TIP: JP2.TIP
- new net N$10: CON2.2, IN1.1
- new net N$12: L1.1, U$4.VBUS
- new net N$13: D3.A, L1.2
- new net N$15: CON2.1, IN1.2
- new net N$16: CON4.2, IN2.1
- new net N$17: CON4.1, IN2.2
- new net N$18: CON1.2, SV1.4
- new net N$19: CON3.2, SV1.5
- new net N$6: JP1.4, JP2.EARTH, SV7.1
- new net N$7: JP1.3, JP2.RING1, SV7.2
- new net N$8: JP1.2, JP2.TIP, SV7.3
- new net N$9: JP1.1, JP2.RING2, SV7.4
- new net THRM: RTHERM.2, SV1.6, THRM.2
- net AOUT: now also SV8.2, SV8.6; no longer SV3.3, SV3.7
- net AOUT1: now also SV6.2, SV6.6; no longer SV5.3, SV5.7
- net GND: now also C2.1, JP3.1, SV1.7, SV6.3, SV8.3, THRM.1, U$4.GND; no longer C3.1, SV1.2, SV1.3, SV3.1, SV3.4, SV5.1, SV5.4, X1.GND
- net N$1: now also SV6.4, SV6.5; no longer SV5.5, SV5.6
- net N$11: now also SV8.4, SV8.5; no longer SV3.5, SV3.6
- net N$14: now also C2.2; no longer C3.2
- net VAIN: now also SV8.1; no longer SV3.2
- net VAIN1: now also SV6.1; no longer SV5.2
- net VBUS: now also D3.C; no longer IC3.VIN, X1.VBUS
- net VCC: now also CON1.1, CON3.1, RTHERM.1
Other:
- note added: "C"
- note added: "O"
- note added: "P"
- note added: "R"
- note added: "Thermistor"
- moved on the sheet: JP2, SV6, SV7

Commit message: update
Parts:
- added C3: 0.1uF, SparkFun:CAP0603-CAP
- added CON5: (no value), pinhead:PINHD-1X2
- added TM1: (no value), adafruit:TRIMPOTTC33X
Connections:
- new net N$20: CON5.1, TM1.A
- new net N$21: C3.2, CON5.2
- new net N$22: C3.1, TM1.S
- net GND: now also TM1.E
Other:
- moved on the sheet: JP1, JP2
Changed lines of the file:
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@@
 <layer number="113" name="IDFDebug" color="7" fill="1" visible="yes" active="yes"/>
 <layer number="116" name="Patch_BOT" color="9" fill="4" visible="no" active="yes"/>
+<layer number="118" name="Rect_Pads" color="7" fill="1" visible="no" active="no"/>
 <layer number="121" name="_tsilk" color="7" fill="1" visible="no" active="yes"/>
 <layer number="122" name="_bsilk" color="7" fill="1" visible="no" active="yes"/>
@@
 <layer number="223" name="223bmp" color="24" fill="1" visible="no" active="no"/>
 <layer number="224" name="224bmp" color="25" fill="1" visible="no" active="no"/>
+<layer number="231" name="Eagle3D_PG1" color="7" fill="1" visible="yes" active="yes"/>
+<layer number="232" name="Eagle3D_PG2" color="7" fill="1" visible="yes" active="yes"/>
+<layer number="233" name="Eagle3D_PG3" color="7" fill="1" visible="yes" active="yes"/>
 <layer number="248" name="Housing" color="7" fill="1" visible="yes" active="yes"/>
 <layer number="249" name="Edge" color="7" fill="1" visible="yes" active="yes"/>
@@
 </variantdefs>
 <classes>
-<class number="0" name="default" width="0.2032" drill="0.3302">
-<clearance class="0" value="0.2032"/>
+<class number="0" name="default" width="0" drill="0">
 </class>
 <class number="1" name="vcc" width="0" drill="0">
@@
 <part name="GND6" library="SparkFun" deviceset="GND" device=""/>
 <part name="RTHERM" library="microbuilder" deviceset="RESISTOR" device="_0603_NOOUT" value="10k"/>
+<part name="CON5" library="pinhead" deviceset="PINHD-1X2" device=""/>
+<part name="C3" library="SparkFun" deviceset="CAP" device="0603-CAP" value="0.1uF"/>
+<part name="GND8" library="supply1" deviceset="GND" device=""/>
+<part name="TM1" library="adafruit" deviceset="TRIMPOT" device="TC33X"/>
 </parts>
 <sheets>
@@
 <instance part="GND2" gate="1" x="-77.47" y="54.356"/>
 <instance part="GND12" gate="1" x="-82.296" y="21.844" rot="MR0"/>
-<instance part="JP2" gate="G$1" x="41.402" y="130.556" smashed="yes" rot="R270">
-<attribute name="NAME" x="46.99" y="135.636" size="1.778" layer="95" rot="R270"/>
-<attribute name="VALUE" x="33.782" y="135.636" size="1.778" layer="96" rot="R270"/>
+<instance part="JP2" gate="G$1" x="35.052" y="139.7" smashed="yes" rot="R270">
+<attribute name="NAME" x="40.64" y="144.78" size="1.778" layer="95" rot="R270"/>
+<attribute name="VALUE" x="27.432" y="144.78" size="1.778" layer="96" rot="R270"/>
 </instance>
 <instance part="CHG2" gate="G$1" x="-46.228" y="21.844" smashed="yes"/>
@@
 <instance part="SV7" gate="1" x="23.368" y="107.188" rot="R90"/>
 <instance part="U$4" gate="G$1" x="-89.154" y="29.464" rot="R180"/>
-<instance part="JP1" gate="A" x="25.908" y="144.78" rot="R90"/>
+<instance part="JP1" gate="A" x="17.018" y="141.224" rot="R90"/>
 <instance part="IN1" gate="G$1" x="-45.212" y="119.634" rot="R90"/>
 <instance part="IN2" gate="G$1" x="7.366" y="121.412" rot="R90"/>
@@
 <instance part="GND6" gate="1" x="-29.464" y="157.48" rot="R270"/>
 <instance part="RTHERM" gate="G$1" x="-5.588" y="157.48" rot="R180"/>
+<instance part="CON5" gate="G$1" x="68.834" y="84.836" rot="R90"/>
+<instance part="C3" gate="G$1" x="68.834" y="71.628" smashed="yes" rot="R180">
+<attribute name="NAME" x="75.692" y="73.533" size="1.778" layer="95" rot="R180"/>
+<attribute name="VALUE" x="78.994" y="70.993" size="1.778" layer="96" rot="R180"/>
+</instance>
+<instance part="GND8" gate="1" x="66.294" y="49.276"/>
+<instance part="TM1" gate="G$1" x="66.294" y="60.198" rot="R180"/>
 </instances>
 <busses>
@@
 <wire x1="-18.288" y1="157.48" x2="-18.288" y2="166.116" width="0.1524" layer="91"/>
 </segment>
+<segment>
+<pinref part="TM1" gate="G$1" pin="E"/>
+<pinref part="GND8" gate="1" pin="GND"/>
+<wire x1="66.294" y1="51.816" x2="66.294" y2="55.118" width="0.1524" layer="91"/>
+</segment>
 </net>
 <net name="VBUS" class="1">
@@
 <pinref part="JP2" gate="G$1" pin="EARTH"/>
 <pinref part="SV7" gate="1" pin="1"/>
-<wire x1="28.448" y1="114.808" x2="46.482" y2="125.476" width="0.1524" layer="91"/>
+<wire x1="28.448" y1="114.808" x2="40.132" y2="134.62" width="0.1524" layer="91"/>
 <pinref part="JP1" gate="A" pin="4"/>
-<wire x1="28.448" y1="114.808" x2="28.448" y2="142.24" width="0.1524" layer="91"/>
+<wire x1="28.448" y1="114.808" x2="19.558" y2="138.684" width="0.1524" layer="91"/>
 <junction x="28.448" y="114.808"/>
 </segment>
@@
 <pinref part="JP2" gate="G$1" pin="RING1"/>
 <pinref part="SV7" gate="1" pin="2"/>
-<wire x1="25.908" y1="114.808" x2="43.942" y2="125.476" width="0.1524" layer="91"/>
+<wire x1="25.908" y1="114.808" x2="37.592" y2="134.62" width="0.1524" layer="91"/>
 <pinref part="JP1" gate="A" pin="3"/>
-<wire x1="25.908" y1="142.24" x2="25.908" y2="114.808" width="0.1524" layer="91"/>
+<wire x1="17.018" y1="138.684" x2="25.908" y2="114.808" width="0.1524" layer="91"/>
 <junction x="25.908" y="114.808"/>
 </segment>
@@
 <pinref part="JP2" gate="G$1" pin="TIP"/>
 <pinref part="SV7" gate="1" pin="3"/>
-<wire x1="23.368" y1="114.808" x2="38.862" y2="125.476" width="0.1524" layer="91"/>
+<wire x1="23.368" y1="114.808" x2="32.512" y2="134.62" width="0.1524" layer="91"/>
 <pinref part="JP1" gate="A" pin="2"/>
-<wire x1="23.368" y1="114.808" x2="23.368" y2="142.24" width="0.1524" layer="91"/>
+<wire x1="23.368" y1="114.808" x2="14.478" y2="138.684" width="0.1524" layer="91"/>
 <junction x="23.368" y="114.808"/>
 </segment>
@@
 <pinref part="JP2" gate="G$1" pin="RING2"/>
 <pinref part="SV7" gate="1" pin="4"/>
-<wire x1="20.828" y1="114.808" x2="36.322" y2="125.476" width="0.1524" layer="91"/>
+<wire x1="20.828" y1="114.808" x2="29.972" y2="134.62" width="0.1524" layer="91"/>
 <pinref part="JP1" gate="A" pin="1"/>
-<wire x1="20.828" y1="114.808" x2="20.828" y2="142.24" width="0.1524" layer="91"/>
+<wire x1="20.828" y1="114.808" x2="11.938" y2="138.684" width="0.1524" layer="91"/>
 <junction x="20.828" y="114.808"/>
 </segment>
@@
 </segment>
 </net>
+<net name="N$20" class="0">
+<segment>
+<pinref part="CON5" gate="G$1" pin="1"/>
+<pinref part="TM1" gate="G$1" pin="A"/>
+<wire x1="66.294" y1="65.278" x2="66.294" y2="82.296" width="0.1524" layer="91"/>
+</segment>
+</net>
+<net name="N$21" class="0">
+<segment>
+<pinref part="CON5" gate="G$1" pin="2"/>
+<pinref part="C3" gate="G$1" pin="2"/>
+<wire x1="68.834" y1="74.168" x2="68.834" y2="82.296" width="0.1524" layer="91"/>
+</segment>
+</net>
+<net name="N$22" class="0">
+<segment>
+<pinref part="TM1" gate="G$1" pin="S"/>
+<wire x1="61.214" y1="60.198" x2="59.182" y2="60.198" width="0.1524" layer="91"/>
+<wire x1="59.182" y1="60.198" x2="59.182" y2="66.548" width="0.1524" layer="91"/>
+<pinref part="C3" gate="G$1" pin="1"/>
+<wire x1="59.182" y1="66.548" x2="68.834" y2="66.548" width="0.1524" layer="91"/>
+</segment>
+</net>

Commit message: update
Parts:
- added JP4: (no value), pinhead:PINHD-1X1
Connections:
- net GND: now also JP4.1
Other:
- moved on the sheet: C1, CON1, CON4, ICB1, JP1, JP2, JP3, RTHERM, SV6, SV7

Commit message: update
Connections:
- net VBUS: now also IC3.VIN
Other:
- moved on the sheet: IC3
Changed lines of the file:
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@@
 <setting verticaltext="up"/>
 </settings>
-<grid distance="0.1" unitdist="inch" unit="inch" style="lines" multiple="1" display="no" altdistance="0.01" altunitdist="inch" altunit="inch"/>
+<grid distance="0.01" unitdist="inch" unit="inch" style="lines" multiple="1" display="no" altdistance="0.01" altunitdist="inch" altunit="inch"/>
 <layers>
 <layer number="1" name="Top" color="4" fill="1" visible="no" active="no"/>
@@
 <instance part="ICB" gate="A" x="-55.88" y="77.47"/>
 <instance part="GND5" gate="1" x="4.572" y="9.144" rot="MR0"/>
-<instance part="IC3" gate="G$1" x="-32.258" y="32.004"/>
+<instance part="IC3" gate="G$1" x="-32.512" y="34.29"/>
 <instance part="BATT" gate="G$1" x="53.594" y="-4.064"/>
 <instance part="J1" gate="G$1" x="-4.318" y="35.814" smashed="yes">
@@
 <instance part="L1" gate="G$1" x="-73.152" y="32.004"/>
 <instance part="D3" gate="G$1" x="-58.674" y="34.544"/>
-<instance part="R1" gate="G$1" x="-46.228" y="29.464" rot="R90"/>
+<instance part="R1" gate="G$1" x="-46.228" y="29.718" rot="R90"/>
 <instance part="C2" gate="G$1" x="-72.39" y="74.93" smashed="yes" rot="R90">
 <attribute name="NAME" x="-70.993" y="71.882" size="1.778" layer="95" rot="R270"/>
@@
 </segment>
 <segment>
-<wire x1="-22.098" y1="29.464" x2="-22.098" y2="11.684" width="0.1524" layer="91"/>
+<wire x1="-22.352" y1="31.75" x2="-22.098" y2="11.684" width="0.1524" layer="91"/>
 <wire x1="-22.098" y1="11.684" x2="-17.018" y2="11.684" width="0.1524" layer="91"/>
 <wire x1="-17.018" y1="21.844" x2="-17.018" y2="11.684" width="0.1524" layer="91"/>
@@
 <pinref part="C1" gate="G$1" pin="1"/>
 <junction x="-10.668" y="73.914"/>
+<junction x="-77.47" y="58.928"/>
 </segment>
 <segment>
@@
 <pinref part="R1" gate="G$1" pin="2"/>
 <pinref part="D3" gate="G$1" pin="C"/>
-<wire x1="-56.134" y1="34.544" x2="-46.228" y2="34.544" width="0.1524" layer="91"/>
+<wire x1="-56.134" y1="34.544" x2="-46.228" y2="34.798" width="0.1524" layer="91"/>
+<wire x1="-46.228" y1="34.798" x2="-42.672" y2="36.83" width="0.1524" layer="91"/>
+<pinref part="IC3" gate="G$1" pin="VIN"/>
+<junction x="-46.228" y="34.798"/>
 </segment>
 </net>
@@
 <net name="VBAT" class="1">
 <segment>
-<wire x1="-22.098" y1="34.544" x2="-9.398" y2="34.544" width="0.1524" layer="91"/>
+<wire x1="-22.352" y1="36.83" x2="-9.398" y2="34.544" width="0.1524" layer="91"/>
 <label x="-20.828" y="34.544" size="1.778" layer="95"/>
 <pinref part="IC3" gate="G$1" pin="VBAT"/>
@@
 <net name="N$3" class="0">
 <segment>
-<wire x1="-22.098" y1="32.004" x2="-17.018" y2="32.004" width="0.1524" layer="91"/>
+<wire x1="-22.352" y1="34.29" x2="-17.018" y2="32.004" width="0.1524" layer="91"/>
 <pinref part="IC3" gate="G$1" pin="PROG"/>
 <pinref part="R2" gate="G$1" pin="2"/>
@@
 </segment>
 </net>
-<net name="VBUS1" class="1">
-<segment>
-<wire x1="-46.228" y1="34.544" x2="-42.418" y2="34.544" width="0.1524" layer="91"/>
-</segment>
-</net>
 <net name="N$5" class="0">
 <segment>
 <wire x1="-46.228" y1="16.764" x2="-42.418" y2="16.764" width="0.1524" layer="91"/>
-<wire x1="-42.418" y1="16.764" x2="-42.418" y2="29.464" width="0.1524" layer="91"/>
+<wire x1="-42.418" y1="16.764" x2="-42.672" y2="31.75" width="0.1524" layer="91"/>
 <pinref part="CHG2" gate="G$1" pin="C"/>
 <pinref part="IC3" gate="G$1" pin="STAT"/>
@@
 <pinref part="CHG2" gate="G$1" pin="A"/>
 <pinref part="R1" gate="G$1" pin="1"/>
-</segment>
-</net>
+<wire x1="-46.228" y1="24.638" x2="-46.228" y2="24.384" width="0.1524" layer="91"/>
+</segment>
+</net>
