File: coqui-v0.2.sch (EAGLE design)
At the start: 33 parts, among them IC3 MCP73831, IC4 MCP1700-33, J1 AYZ0202

Commit message: update
Parts:
- renumbered CHG2 to CHG, ICB to 555A, ICB1 to 555B
Changed lines of the file:
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@@
 <setting verticaltext="up"/>
 </settings>
-<grid distance="0.01" unitdist="inch" unit="inch" style="lines" multiple="1" display="no" altdistance="0.01" altunitdist="inch" altunit="inch"/>
+<grid distance="0.1" unitdist="inch" unit="inch" style="lines" multiple="1" display="no" altdistance="0.01" altunitdist="inch" altunit="inch"/>
 <layers>
 <layer number="1" name="Top" color="4" fill="1" visible="no" active="no"/>
@@
 </classes>
 <parts>
-<part name="ICB" library="adafruit" deviceset="*555" device="D" technology="LM"/>
+<part name="555A" library="adafruit" deviceset="*555" device="D" technology="LM"/>
 <part name="GND5" library="supply1" deviceset="GND" device=""/>
 <part name="IC3" library="SparkFunNew" deviceset="MCP73831" device=""/>
@@
 <part name="GND12" library="supply1" deviceset="GND" device=""/>
 <part name="JP2" library="SparkFun-Connectors" deviceset="AUDIO-JACK3" device=""/>
-<part name="CHG2" library="led" deviceset="LED" device="CHIPLED_0805" value="0805"/>
-<part name="ICB1" library="adafruit" deviceset="*555" device="D" technology="LM"/>
+<part name="CHG" library="led" deviceset="LED" device="CHIPLED_0805" value="0805"/>
+<part name="555B" library="adafruit" deviceset="*555" device="D" technology="LM"/>
 <part name="GND1" library="supply1" deviceset="GND" device=""/>
 <part name="SV7" library="con-lstb" deviceset="MA04-1" device=""/>
@@
 </plain>
 <instances>
-<instance part="ICB" gate="A" x="-55.88" y="77.47"/>
+<instance part="555A" gate="A" x="-55.88" y="77.47"/>
 <instance part="GND5" gate="1" x="4.572" y="9.144" rot="MR0"/>
 <instance part="IC3" gate="G$1" x="-32.512" y="34.29"/>
@@
 <attribute name="VALUE" x="37.592" y="144.78" size="1.778" layer="96" rot="R270"/>
 </instance>
-<instance part="CHG2" gate="G$1" x="-46.228" y="21.844" smashed="yes"/>
-<instance part="ICB1" gate="A" x="10.922" y="76.454"/>
+<instance part="CHG" gate="G$1" x="-46.228" y="21.844" smashed="yes"/>
+<instance part="555B" gate="A" x="10.922" y="76.454"/>
 <instance part="GND1" gate="1" x="-10.668" y="61.214"/>
 <instance part="SV7" gate="1" x="33.528" y="107.188" rot="R90"/>
@@
 <pinref part="GND2" gate="1" pin="GND"/>
 <wire x1="-77.47" y1="56.896" x2="-77.47" y2="58.928" width="0.1524" layer="91"/>
-<pinref part="ICB" gate="A" pin="GND"/>
+<pinref part="555A" gate="A" pin="GND"/>
 <wire x1="-77.47" y1="58.928" x2="-77.47" y2="69.85" width="0.1524" layer="91"/>
 <wire x1="-66.04" y1="69.85" x2="-77.47" y2="69.85" width="0.1524" layer="91"/>
@@
 <pinref part="GND1" gate="1" pin="GND"/>
 <wire x1="-10.668" y1="63.754" x2="-10.668" y2="66.04" width="0.1524" layer="91"/>
-<pinref part="ICB1" gate="A" pin="GND"/>
+<pinref part="555B" gate="A" pin="GND"/>
 <wire x1="-10.668" y1="66.04" x2="-10.668" y2="68.834" width="0.1524" layer="91"/>
 <wire x1="0.762" y1="68.834" x2="-10.668" y2="68.834" width="0.1524" layer="91"/>
@@
 <net name="AOUT" class="0">
 <segment>
-<pinref part="ICB" gate="A" pin="Q"/>
+<pinref part="555A" gate="A" pin="Q"/>
 <wire x1="-45.72" y1="85.09" x2="-41.91" y2="85.09" width="0.1524" layer="91"/>
 <wire x1="-41.91" y1="85.09" x2="-41.91" y2="97.79" width="0.1524" layer="91"/>
@@
 <net name="N$11" class="0">
 <segment>
-<pinref part="ICB" gate="A" pin="THR"/>
+<pinref part="555A" gate="A" pin="THR"/>
 <wire x1="-45.72" y1="74.93" x2="-39.116" y2="74.93" width="0.1524" layer="91"/>
 <wire x1="-39.116" y1="74.93" x2="-39.116" y2="91.44" width="0.1524" layer="91"/>
-<pinref part="ICB" gate="A" pin="TR"/>
+<pinref part="555A" gate="A" pin="TR"/>
 <wire x1="-39.116" y1="91.44" x2="-64.77" y2="91.44" width="0.1524" layer="91"/>
 <wire x1="-64.77" y1="91.44" x2="-66.04" y2="91.44" width="0.1524" layer="91"/>
@@
 <net name="N$14" class="0">
 <segment>
-<pinref part="ICB" gate="A" pin="CV"/>
+<pinref part="555A" gate="A" pin="CV"/>
 <wire x1="-69.85" y1="74.93" x2="-66.04" y2="74.93" width="0.1524" layer="91"/>
 <pinref part="C2" gate="G$1" pin="2"/>
@@
 <net name="VAIN" class="0">
 <segment>
-<pinref part="ICB" gate="A" pin="V+"/>
+<pinref part="555A" gate="A" pin="V+"/>
 <wire x1="-45.72" y1="69.85" x2="-42.164" y2="69.85" width="0.1524" layer="91"/>
 <wire x1="-74.93" y1="101.6" x2="-74.93" y2="80.01" width="0.1524" layer="91"/>
-<pinref part="ICB" gate="A" pin="R"/>
+<pinref part="555A" gate="A" pin="R"/>
 <wire x1="-74.93" y1="80.01" x2="-68.834" y2="80.01" width="0.1524" layer="91"/>
 <wire x1="-68.834" y1="80.01" x2="-66.04" y2="80.01" width="0.1524" layer="91"/>
@@
 <wire x1="-46.228" y1="16.764" x2="-42.418" y2="16.764" width="0.1524" layer="91"/>
 <wire x1="-42.418" y1="16.764" x2="-42.672" y2="31.75" width="0.1524" layer="91"/>
-<pinref part="CHG2" gate="G$1" pin="C"/>
+<pinref part="CHG" gate="G$1" pin="C"/>
 <pinref part="IC3" gate="G$1" pin="STAT"/>
 </segment>
@@
 <net name="AOUT1" class="0">
 <segment>
-<pinref part="ICB1" gate="A" pin="Q"/>
+<pinref part="555B" gate="A" pin="Q"/>
 <wire x1="21.082" y1="84.074" x2="24.892" y2="84.074" width="0.1524" layer="91"/>
 <wire x1="24.892" y1="84.074" x2="24.892" y2="96.774" width="0.1524" layer="91"/>
@@
 <net name="N$1" class="0">
 <segment>
-<pinref part="ICB1" gate="A" pin="THR"/>
+<pinref part="555B" gate="A" pin="THR"/>
 <wire x1="21.082" y1="73.914" x2="27.686" y2="73.914" width="0.1524" layer="91"/>
 <wire x1="27.686" y1="73.914" x2="27.686" y2="90.424" width="0.1524" layer="91"/>
-<pinref part="ICB1" gate="A" pin="TR"/>
+<pinref part="555B" gate="A" pin="TR"/>
 <wire x1="27.686" y1="90.424" x2="2.032" y2="90.424" width="0.1524" layer="91"/>
 <wire x1="2.032" y1="90.424" x2="0.762" y2="90.424" width="0.1524" layer="91"/>
@@
 <net name="VAIN1" class="0">
 <segment>
-<pinref part="ICB1" gate="A" pin="V+"/>
+<pinref part="555B" gate="A" pin="V+"/>
 <wire x1="21.082" y1="68.834" x2="24.638" y2="68.834" width="0.1524" layer="91"/>
 <wire x1="-8.128" y1="101.346" x2="-8.128" y2="78.994" width="0.1524" layer="91"/>
-<pinref part="ICB1" gate="A" pin="R"/>
+<pinref part="555B" gate="A" pin="R"/>
 <wire x1="-8.128" y1="78.994" x2="-2.032" y2="78.994" width="0.1524" layer="91"/>
 <wire x1="-2.032" y1="78.994" x2="0.762" y2="78.994" width="0.1524" layer="91"/>
@@
 <net name="N$2" class="0">
 <segment>
-<pinref part="ICB1" gate="A" pin="CV"/>
+<pinref part="555B" gate="A" pin="CV"/>
 <wire x1="-3.048" y1="73.914" x2="0.762" y2="73.914" width="0.1524" layer="91"/>
 <pinref part="C1" gate="G$1" pin="2"/>
@@
 <net name="N$4" class="0">
 <segment>
-<pinref part="CHG2" gate="G$1" pin="A"/>
+<pinref part="CHG" gate="G$1" pin="A"/>
 <pinref part="R1" gate="G$1" pin="1"/>
 <wire x1="-46.228" y1="24.638" x2="-46.228" y2="24.384" width="0.1524" layer="91"/>

Commit message: update
Connections:
- net THRM: now also SV1.1; no longer SV1.6
- net VCC: now also SV1.6; no longer SV1.1
Changed lines of the file:
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@@
 <setting verticaltext="up"/>
 </settings>
-<grid distance="0.1" unitdist="inch" unit="inch" style="lines" multiple="1" display="no" altdistance="0.01" altunitdist="inch" altunit="inch"/>
+<grid distance="0.01" unitdist="inch" unit="inch" style="lines" multiple="1" display="no" altdistance="0.01" altunitdist="inch" altunit="inch"/>
 <layers>
 <layer number="1" name="Top" color="4" fill="1" visible="no" active="no"/>
@@
 <instance part="GND3" gate="1" x="-49.022" y="132.08"/>
 <instance part="P+6" gate="VCC" x="31.75" y="34.544"/>
-<instance part="P+1" gate="VCC" x="-72.644" y="140.462"/>
+<instance part="P+1" gate="VCC" x="-39.624" y="140.462"/>
 <instance part="P+2" gate="VCC" x="-96.774" y="116.078"/>
 <instance part="P+3" gate="VCC" x="-29.972" y="115.824"/>
@@
 </segment>
 <segment>
-<pinref part="SV1" gate="1" pin="1"/>
-<pinref part="P+1" gate="VCC" pin="VCC"/>
-<wire x1="-72.644" y1="137.922" x2="-64.262" y2="137.922" width="0.1524" layer="91"/>
-</segment>
-<segment>
 <pinref part="CON1" gate="G$1" pin="1"/>
 <pinref part="P+2" gate="VCC" pin="VCC"/>
@@
 <wire x1="9.652" y1="157.48" x2="17.272" y2="157.48" width="0.1524" layer="91"/>
 <pinref part="RTHERM" gate="G$1" pin="1"/>
+</segment>
+<segment>
+<pinref part="SV1" gate="1" pin="6"/>
+<pinref part="P+1" gate="VCC" pin="VCC"/>
+<wire x1="-51.562" y1="137.922" x2="-39.624" y2="137.922" width="0.1524" layer="91"/>
 </segment>
 </net>
@@
 <junction x="-5.588" y="157.48"/>
 <wire x1="-5.588" y1="157.48" x2="-5.588" y2="135.89" width="0.1524" layer="91"/>
-<pinref part="SV1" gate="1" pin="6"/>
-<wire x1="-5.588" y1="135.89" x2="-51.562" y2="135.89" width="0.1524" layer="91"/>
-<wire x1="-51.562" y1="135.89" x2="-51.562" y2="137.922" width="0.1524" layer="91"/>
+<wire x1="-5.588" y1="135.89" x2="-64.262" y2="135.89" width="0.1524" layer="91"/>
 <pinref part="RTHERM" gate="G$1" pin="2"/>
-</segment>
-</net>
+<pinref part="SV1" gate="1" pin="1"/>
+<wire x1="-64.262" y1="135.89" x2="-64.262" y2="137.922" width="0.1524" layer="91"/>
+</segment>
+</net>
